File: Design Files/Exploding Capacitors Lab/poorUSBadapter/V1I1/poorUSBadapter.sch (EAGLE design)
At the start: 12 parts

Commit message: V1I1 is ready
Parts:
- removed S1: SWITCH-MOMENTARY-2SMD-1101NE, SparkFun-Electromechanical:SWITCH-MOMENTARY-2SMD-1101NE
- added BOOT: SWITCH-MOMENTARY-2SMD-1101NE, SparkFun-Electromechanical:SWITCH-MOMENTARY-2SMD-1101NE
- JP1: device adafruit:PINHD-1X1 -> pinhead:PINHD-1X1
- renumbered USB1 to USB
Connections:
- net DIO7: now also BOOT.2; no longer S1.2
- net GND: now also BOOT.1; no longer S1.1
Other:
- note added: "Exploding Capacitors Lab http://fryco.github.io/poorSUBadapter/"
- note added: "V1I1"
- moved on the sheet: JP1, SJ1, U$1
Changed lines of the file:
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@@
 <setting verticaltext="up"/>
 </settings>
-<grid distance="0.1" unitdist="inch" unit="inch" style="lines" multiple="1" display="yes" altdistance="0.01" altunitdist="inch" altunit="inch"/>
+<grid distance="0.1" unitdist="inch" unit="inch" style="lines" multiple="1" display="no" altdistance="0.01" altunitdist="inch" altunit="inch"/>
 <layers>
 <layer number="1" name="Top" color="4" fill="1" visible="no" active="no"/>
@@
 </classes>
 <parts>
-<part name="FRAME1" library="frames" deviceset="A4L-LOC" device=""/>
 <part name="GND1" library="supply1" deviceset="GND" device=""/>
 <part name="P+1" library="supply1" deviceset="VCC" device=""/>
-<part name="USB1" library="dp_devices" deviceset="CON-USB-F" device="-MINI-B"/>
+<part name="USB" library="dp_devices" deviceset="CON-USB-F" device="-MINI-B"/>
 <part name="GND2" library="supply1" deviceset="GND" device=""/>
 <part name="GND3" library="supply1" deviceset="GND" device=""/>
@@
 <part name="R4" library="SparkFun-Passives" deviceset="RESISTOR" device="0805-RES" value="68R"/>
 <part name="GND4" library="supply1" deviceset="GND" device=""/>
-<part name="S1" library="SparkFun-Electromechanical" deviceset="SWITCH-MOMENTARY-2" device="SMD-1101NE"/>
+<part name="BOOT" library="SparkFun-Electromechanical" deviceset="SWITCH-MOMENTARY-2" device="SMD-1101NE"/>
 <part name="GND5" library="supply1" deviceset="GND" device=""/>
-<part name="SJ1" library="SparkFun-Passives" deviceset="JUMPER-PAD-3-NO" device="FULL_BOX_SILK"/>
-<part name="P+2" library="supply1" deviceset="VCC" device=""/>
-<part name="JP1" library="adafruit" deviceset="PINHD-1X1" device=""/>
 <part name="D3" library="diode" deviceset="DIODE-" device="MICROMELF-W" value="3V6"/>
 <part name="D4" library="diode" deviceset="DIODE-" device="MICROMELF-W" value="3V6"/>
@@
 <part name="JP2" library="adafruit" deviceset="PINHD-1X8" device="BIG"/>
 <part name="GND6" library="supply1" deviceset="GND" device=""/>
+<part name="SJ1" library="SparkFun-Passives" deviceset="JUMPER-PAD-3-NO" device="FULL_BOX_SILK"/>
+<part name="JP1" library="pinhead" deviceset="PINHD-1X1" device=""/>
+<part name="P+2" library="supply1" deviceset="VCC" device=""/>
+<part name="FRAME2" library="frames" deviceset="DINA4_L" device=""/>
 </parts>
 <sheets>
 <sheet>
 <plain>
+<text x="164.465" y="26.67" size="2.54" layer="91">Exploding Capacitors Lab
+http://fryco.github.io/poorSUBadapter/</text>
+<text x="259.715" y="7.62" size="2.54" layer="91" rot="MR0">V1I1</text>
 </plain>
 <instances>
-<instance part="FRAME1" gate="G$1" x="0" y="0"/>
 <instance part="GND1" gate="1" x="93.98" y="55.88"/>
 <instance part="P+1" gate="VCC" x="106.68" y="93.98"/>
-<instance part="USB1" gate="USB" x="43.18" y="76.2"/>
+<instance part="USB" gate="USB" x="43.18" y="76.2"/>
 <instance part="GND2" gate="1" x="73.66" y="55.88"/>
 <instance part="GND3" gate="1" x="83.82" y="55.88"/>
@@
 <instance part="R4" gate="G$1" x="124.46" y="68.58"/>
 <instance part="GND4" gate="1" x="106.68" y="55.88"/>
-<instance part="S1" gate="G$1" x="63.5" y="109.22" rot="R90"/>
-<instance part="GND5" gate="1" x="63.5" y="99.06"/>
-<instance part="SJ1" gate="G$1" x="132.08" y="106.68" rot="R180"/>
-<instance part="P+2" gate="VCC" x="139.7" y="111.76"/>
-<instance part="JP1" gate="G$1" x="119.38" y="114.3" rot="R180"/>
+<instance part="BOOT" gate="G$1" x="78.74" y="132.08" rot="R90"/>
+<instance part="GND5" gate="1" x="78.74" y="121.92"/>
 <instance part="D3" gate="G$1" x="73.66" y="63.5" rot="R90"/>
 <instance part="D4" gate="G$1" x="83.82" y="63.5" rot="R90"/>
-<instance part="U$1" gate="G$1" x="218.44" y="91.44"/>
+<instance part="U$1" gate="G$1" x="203.2" y="73.66"/>
 <instance part="JP2" gate="G$1" x="180.34" y="76.2"/>
-<instance part="GND6" gate="1" x="200.66" y="83.82"/>
+<instance part="GND6" gate="1" x="187.96" y="55.88"/>
+<instance part="SJ1" gate="G$1" x="172.72" y="144.78" rot="R180"/>
+<instance part="JP1" gate="G$1" x="160.02" y="154.94" rot="R180"/>
+<instance part="P+2" gate="VCC" x="180.34" y="149.86"/>
+<instance part="FRAME2" gate="G$1" x="0" y="0"/>
+<instance part="FRAME2" gate="G$2" x="162.56" y="0"/>
 </instances>
 <busses>
@@
 <net name="USB_P" class="0">
 <segment>
-<pinref part="USB1" gate="USB" pin="D+"/>
+<pinref part="USB" gate="USB" pin="D+"/>
 <wire x1="48.26" y1="73.66" x2="73.66" y2="73.66" width="0.1524" layer="91"/>
 <wire x1="73.66" y1="73.66" x2="73.66" y2="66.04" width="0.1524" layer="91"/>
@@
 <net name="USB_N" class="0">
 <segment>
-<pinref part="USB1" gate="USB" pin="D-"/>
+<pinref part="USB" gate="USB" pin="D-"/>
 <wire x1="48.26" y1="76.2" x2="83.82" y2="76.2" width="0.1524" layer="91"/>
 <wire x1="83.82" y1="76.2" x2="83.82" y2="66.04" width="0.1524" layer="91"/>
@@
 <pinref part="GND1" gate="1" pin="GND"/>
 <wire x1="93.98" y1="58.42" x2="93.98" y2="81.28" width="0.1524" layer="91"/>
-<pinref part="USB1" gate="USB" pin="GND"/>
+<pinref part="USB" gate="USB" pin="GND"/>
 <wire x1="93.98" y1="81.28" x2="48.26" y2="81.28" width="0.1524" layer="91"/>
 </segment>
@@
 </segment>
 <segment>
-<pinref part="S1" gate="G$1" pin="1"/>
-<wire x1="63.5" y1="104.14" x2="63.5" y2="101.6" width="0.1524" layer="91"/>
+<pinref part="BOOT" gate="G$1" pin="1"/>
+<wire x1="78.74" y1="127" x2="78.74" y2="124.46" width="0.1524" layer="91"/>
 <pinref part="GND5" gate="1" pin="GND"/>
 </segment>
@@
 <pinref part="U$1" gate="G$1" pin="7"/>
 <pinref part="GND6" gate="1" pin="GND"/>
-<wire x1="215.9" y1="86.36" x2="200.66" y2="86.36" width="0.1524" layer="91"/>
+<wire x1="200.66" y1="68.58" x2="187.96" y2="68.58" width="0.1524" layer="91"/>
+<wire x1="187.96" y1="68.58" x2="187.96" y2="58.42" width="0.1524" layer="91"/>
 </segment>
 <segment>
@@
 <segment>
 <pinref part="SJ1" gate="G$1" pin="2"/>
-<wire x1="137.16" y1="106.68" x2="139.7" y2="106.68" width="0.1524" layer="91"/>
-<wire x1="139.7" y1="106.68" x2="139.7" y2="109.22" width="0.1524" layer="91"/>
+<wire x1="177.8" y1="144.78" x2="180.34" y2="144.78" width="0.1524" layer="91"/>
+<wire x1="180.34" y1="144.78" x2="180.34" y2="147.32" width="0.1524" layer="91"/>
 <pinref part="P+2" gate="VCC" pin="VCC"/>
 </segment>
@@
 <net name="DIO7" class="0">
 <segment>
-<pinref part="S1" gate="G$1" pin="2"/>
-<wire x1="63.5" y1="114.3" x2="63.5" y2="116.84" width="0.1524" layer="91"/>
-<wire x1="63.5" y1="116.84" x2="68.58" y2="116.84" width="0.1524" layer="91"/>
-<label x="68.58" y="116.84" size="1.778" layer="95" xref="yes"/>
+<pinref part="BOOT" gate="G$1" pin="2"/>
+<wire x1="78.74" y1="137.16" x2="78.74" y2="139.7" width="0.1524" layer="91"/>
+<wire x1="78.74" y1="139.7" x2="83.82" y2="139.7" width="0.1524" layer="91"/>
+<label x="83.82" y="139.7" size="1.778" layer="95" xref="yes"/>
 </segment>
 <segment>
@@
 </segment>
 </net>
-<net name="N$3" class="0">
-<segment>
-<pinref part="SJ1" gate="G$1" pin="3"/>
-<wire x1="132.08" y1="111.76" x2="132.08" y2="114.3" width="0.1524" layer="91"/>
-<wire x1="132.08" y1="114.3" x2="121.92" y2="114.3" width="0.1524" layer="91"/>
-<pinref part="JP1" gate="G$1" pin="1"/>
-<wire x1="121.92" y1="114.3" x2="124.46" y2="114.3" width="0.1524" layer="91"/>
-</segment>
-</net>
 <net name="DIO3" class="0">
-<segment>
-<pinref part="SJ1" gate="G$1" pin="1"/>
-<wire x1="132.08" y1="101.6" x2="132.08" y2="99.06" width="0.1524" layer="91"/>
-<wire x1="132.08" y1="99.06" x2="124.46" y2="99.06" width="0.1524" layer="91"/>
-<label x="124.46" y="99.06" size="1.778" layer="95" rot="R180" xref="yes"/>
-</segment>
 <segment>
 <pinref part="JP2" gate="G$1" pin="4"/>
 <wire x1="177.8" y1="76.2" x2="170.18" y2="76.2" width="0.1524" layer="91"/>
 <label x="170.18" y="76.2" size="1.778" layer="95" rot="R180" xref="yes"/>
+</segment>
+<segment>
+<pinref part="SJ1" gate="G$1" pin="1"/>
+<wire x1="172.72" y1="139.7" x2="172.72" y2="134.62" width="0.1524" layer="91"/>
+<wire x1="172.72" y1="134.62" x2="162.56" y2="134.62" width="0.1524" layer="91"/>
+<label x="162.56" y="134.62" size="1.778" layer="95" rot="R180" xref="yes"/>
+</segment>
+</net>
+<net name="N$1" class="0">
+<segment>
+<pinref part="JP1" gate="G$1" pin="1"/>
+<wire x1="162.56" y1="154.94" x2="172.72" y2="154.94" width="0.1524" layer="91"/>
+<pinref part="SJ1" gate="G$1" pin="3"/>
+<wire x1="172.72" y1="154.94" x2="172.72" y2="149.86" width="0.1524" layer="91"/>
 </segment>
 </net>
@@
 </schematic>
 </drawing>
+<compatibility>
+<note version="6.3" minversion="6.2.2" severity="warning">
+Since Version 6.2.2 text objects can contain more than one line,
+which will not be processed correctly with this version.
+</note>
+</compatibility>
 </eagle>
